Commit message: initial commit

File: urdf/4WD.xacro (robot description, xacro)
@@ -156,5 +156,5 @@
 </joint>
 <joint name="Rigid28" type="fixed">
-  <origin rpy="0 0 0" xyz="0.179596 8e-06 0.299905"/>
+  <origin rpy="0 0 3.14" xyz="0.179596 8e-06 0.299905"/>
   <parent link="base_link"/>
   <child link="lidar_base_1"/>
